File: electronics/blandpanel/blandpanel.kicad_pcb (KiCad board)
At the start: 2 copper layers, 13 parts, among them J1 Barrel_Jack, M1 Motor_Servo, Q1 TIP120, Q2 NPN, U1 Pico, U2 LM1085-5.0

Commit message: Updates for semi-final design
Parts:
- removed U2: LM1085-5.0, Package_TO_SOT_THT:TO-220-3_Vertical
- added U3: LM2576HVT-5, Package_TO_SOT_THT:TO-220-5_Vertical, F.Cu at (159.4, 137.4)
- D2: value LED_Series -> 12V LED Strip
- M1: value Motor_Servo -> 5V PWM Servo
- moved M1 3.50 mm to (154.0, 115.5)
- moved D1 3.42 mm to (152.9, 121.5)
- turned Q2 to 90 degrees
- renumbered R3 to RSENSE1
Connections:
- net Net-(D1-A) renamed +5V
- J1 pad 1: GND -> VCC +12V
- J1 pad 2: VCC +12V -> GND
- R1 pad 1: Net-(U1-GPIO15) -> Net-(Q1-B)
- R1 pad 2: Net-(Q1-B) -> Net-(U1-GPIO15)
- U1 pad 19: unconnected-(U1-GPIO14-Pad19) -> Net-(U1-GPIO14)
Routing:
- net Net-(U1-GPIO14): track 0.00 -> 34.6 mm
- net +5V: track 60.7 -> 70.0 mm
- net VCC +12V: track 135.9 -> 126.9 mm
- net Net-(Q2-B): track 6.46 -> 12.8 mm
- net Net-(D1-K): track 67.1 -> 70.5 mm
- net Net-(Q1-B): track 17.5 -> 15.0 mm
- net Net-(M1-PWM): track 29.8 -> 32.1 mm
- net Net-(M1-ANG): track 48.8 -> 47.5 mm
- net Net-(D2-K): track 18.2 -> 19.4 mm
Other:
- board text added: "+"
- board text added: "-"
- board text added: "ANG"
- board text added: "PWM"
