File: electronics/blandpanel/blandpanel.kicad_sch (KiCad schematic)
At the start: 13 parts, among them J1 Barrel_Jack, M1 Motor_Servo, Q1 TIP120, Q2 NPN, U1 Pico, U2 LM1085-5.0

Commit message: Updates for semi-final design
Parts:
- removed U2: LM1085-5.0, Package_TO_SOT_THT:TO-220-3_Vertical, symbol Regulator_Linear:LM1085-5.0
- added R4: 1k, symbol Device:R_US
- added U3: LM2576HVT-5, Package_TO_SOT_THT:TO-220-5_Vertical, symbol Regulator_Switching:LM2576HVT-5
- D2: value LED_Series -> 12V LED Strip
- M1: value Motor_Servo -> 5V PWM Servo
- renumbered R3 to RSENSE1
Connections:
- net GND: now also J1.2, R4.2, U3.3 (GND); no longer J1.1
- net VCC +12V: now also J1.1, U3.1 (VIN); no longer J1.2
- net at R1.1: now also Q1.1 (B), Q2.1 (C); no longer U1.20 (GPIO15)
- net +5V: now reaches C1.1, D1.2 (A), M1.2 (+)
- net +5V: now also U3.2 (OUT), U3.4 (FB)
- net at U1.19 (GPIO14): now also R4.1, U3.5 (~{ON}/OFF)
- new net: R1.2, U1.20 (GPIO15)
- no-connect marks 0 -> 1
Other:
- moved on the sheet: C1, C2, D1, D2, J1, M1, Q1, Q2, R1, R2, RSENSE1, U1
